File: embedded/board-design/esp32-main/esp32-main.kicad_pcb (KiCad board)
At the start: 2 copper layers, 70.5 x 135.5 mm, 81 parts, among them J1 Conn_ARM_JTAG_SWD_10, J2 Conn_01x08_Socket, J3 Conn_01x08_Socket, J4 0473460001, J5 Conn_01x03_Socket, Q1 BC817, Q2 BC817, Q3 FDN340P, Q4 FMMT720TA, Q5 FDN340P, Q6 FDN340P, U1 ESP32-WROVER-E, U2 BD48ExxG, U3 FT231XS, U4 TPS61090, U5 LTC4054ES5-4.2

Commit message: [bike-embedded-app]
Signed-off-by: Nicolae-Andrei Vasile <vasilenicolaeandrei@gmail.com>
Parts:
- added J6: Conn_01x02_Socket, Connector_PinHeader_1.27mm:PinHeader_1x02_P1.27mm_Vertical, F.Cu at (141.0, 108.0)
- added J7: Conn_01x03_Socket, Connector_Phoenix_MC:PhoenixContact_MC_1,5_3-G-3.81_1x03_P3.81mm_Horizontal, F.Cu at (157.2, 147.1)
- J5: value Conn_01x03_Socket -> Conn_01x02_Socket; footprint Connector_Phoenix_MC:PhoenixContact_MC_1,5_3-G-3.81_1x03_P3.81mm_Horizontal -> Connector_PinHeader_1.27mm:PinHeader_1x02_P1.27mm_Vertical
- moved J5 39.6 mm to (118.0, 142.0)
Connections:
- net Net-(D4-K) renamed /power-supply/VBAT_TEST
- J5 pad 1: /battery/ALT -> VBUS
Routing:
- net /power-supply/VBAT_TEST: track 2.18 -> 5.70 mm
